Commit message: 添加手动模式

File: workspace/src/franka_description/robots/common/franka_arm.ros2_control.xacro (robot description, xacro)
@@ -51,4 +51,25 @@
         </joint>
       </xacro:macro>
+      <!-- Gazebo's ros2_control plugin only synchronizes mimic joints that
+           are explicitly listed in the hardware description.  This is kept
+           separate from configure_joint so ordinary arm joints never receive
+           an empty/default "mimic" parameter. -->
+      <xacro:macro name="configure_mimic_joint" params="joint_name initial_position mimic_joint">
+        <joint name="${joint_name}">
+          <param name="mimic">${mimic_joint}</param>
+          <param name="multiplier">1.0</param>
+          <command_interface name="position"/>
+          <command_interface name="velocity"/>
+          <xacro:if value="${gazebo == 0 or gazebo_effort == 1}">
+            <command_interface name="effort"/>
+          </xacro:if>
+          <state_interface name="position">
+            <param name="initial_value">${initial_position}</param>
+          </state_interface>
+          <state_interface name="velocity"/>
+            <param name="initial_value">0.0</param>
+          <state_interface name="effort"/>
+        </joint>
+      </xacro:macro>
       <xacro:configure_joint joint_name="${arm_prefix}${arm_id}_joint1" initial_position="0.0"/>
       <xacro:configure_joint joint_name="${arm_prefix}${arm_id}_joint2" initial_position="${-pi/4}"/>
@@ -60,4 +81,10 @@
       <xacro:if value="${gazebo and hand}">
         <xacro:configure_joint joint_name="${arm_prefix}${arm_id}_finger_joint1" initial_position="0.0" />
+        <!-- Register the second finger as a Gazebo hardware mimic.  Keeping
+             it out of ros2_control left one visual/physical finger static. -->
+        <xacro:configure_mimic_joint
+          joint_name="${arm_prefix}${arm_id}_finger_joint2"
+          initial_position="0.0"
+          mimic_joint="${arm_prefix}${arm_id}_finger_joint1" />
       </xacro:if>
       <xacro:macro name="general_purpose_io" params="prefix command_interface index">
